Commit message: created_nervous_system_of_swarm

File: install/turtlebot3_gazebo/share/turtlebot3_gazebo/urdf/my_bot.urdf (robot description, URDF)
Before this commit: robot turtlebot3_waffle_pi, 11 links, 10 joints
Links:
- removed link bot_2/base_footprint
- removed link bot_2/base_link
- removed link bot_2/base_scan
- removed link bot_2/camera_link
- removed link bot_2/camera_rgb_frame
- removed link bot_2/camera_rgb_optical_frame
- removed link bot_2/caster_back_left_link
- removed link bot_2/caster_back_right_link
- removed link bot_2/imu_link
- removed link bot_2/wheel_left_link
- removed link bot_2/wheel_right_link
- added link bot_1/base_footprint
- added link bot_1/base_link, mass 1.3729096e+00; collision box size=0.266 0.266 0.094; visual mesh filename=file:///home/pacman/turtlebot3_ws/install/turtlebot3_xacro/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 scale=0.001 0.001 0.001
- added link bot_1/base_scan, mass 0.114; collision cylinder length=0.0315 radius=0.055; visual mesh filename=file:///home/pacman/turtlebot3_ws/install/turtlebot3_xacro/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 scale=0.001 0.001 0.001
- added link bot_1/camera_link; collision box size=0.015 0.030 0.027
- added link bot_1/camera_rgb_frame
- added link bot_1/camera_rgb_optical_frame
- added link bot_1/caster_back_left_link, mass 0.005; collision sphere radius=0.009
- added link bot_1/caster_back_right_link, mass 0.005; collision sphere radius=0.009
- added link bot_1/imu_link, mass 0.001
- added link bot_1/wheel_left_link, mass 2.8498940e-02; collision cylinder length=0.018 radius=0.033; visual mesh filename=file:///home/pacman/turtlebot3_ws/install/turtlebot3_xacro/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 scale=0.001 0.001 0.001
- added link bot_1/wheel_right_link, mass 2.8498940e-02; collision cylinder length=0.018 radius=0.033; visual mesh filename=file:///home/pacman/turtlebot3_ws/install/turtlebot3_xacro/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 scale=0.001 0.001 0.001
Joints:
- joint base_joint: child bot_2/base_link -> bot_1/base_link; parent bot_2/base_footprint -> bot_1/base_footprint
- joint camera_joint: child bot_2/camera_link -> bot_1/camera_link; parent bot_2/base_link -> bot_1/base_link
- joint camera_rgb_joint: child bot_2/camera_rgb_frame -> bot_1/camera_rgb_frame; parent bot_2/camera_link -> bot_1/camera_link
- joint camera_rgb_optical_joint: child bot_2/camera_rgb_optical_frame -> bot_1/camera_rgb_optical_frame; parent bot_2/camera_rgb_frame -> bot_1/camera_rgb_frame
- joint caster_back_left_joint: child bot_2/caster_back_left_link -> bot_1/caster_back_left_link; parent bot_2/base_link -> bot_1/base_link
- joint caster_back_right_joint: child bot_2/caster_back_right_link -> bot_1/caster_back_right_link; parent bot_2/base_link -> bot_1/base_link
- joint imu_joint: child bot_2/imu_link -> bot_1/imu_link; parent bot_2/base_link -> bot_1/base_link
- joint scan_joint: child bot_2/base_scan -> bot_1/base_scan; parent bot_2/base_link -> bot_1/base_link
- joint wheel_left_joint: child bot_2/wheel_left_link -> bot_1/wheel_left_link; parent bot_2/base_link -> bot_1/base_link
- joint wheel_right_joint: child bot_2/wheel_right_link -> bot_1/wheel_right_link; parent bot_2/base_link -> bot_1/base_link

File: install/turtlebot3_xacro/share/turtlebot3_xacro/urdf/common_properties.xacro (robot description, xacro)
@@ -37,5 +37,5 @@
  </xacro:if>
  <xacro:macro name="mesh" params="mesh">
-     <mesh filename="package://turtlebot3_xacro/meshes/${mesh}" scale="0.001 0.001 0.001"/>
+     <mesh filename="file://$(find turtlebot3_xacro)/meshes/${mesh}" scale="0.001 0.001 0.001"/>
  </xacro:macro>
 </robot>

File: install/turtlebot3_xacro/share/turtlebot3_xacro/urdf/turtlebot3_gazebo.xacro (robot description, xacro)
@@ -24,7 +24,5 @@
     <sensor name="tb3_imu" type="imu">
         <always_on>true</always_on>
-        <update_rate>50</update_rate>
-        <topic>$(arg prefix)imu</topic>
-        <gz_frame_id>$(arg prefix)imu_link</gz_frame_id>
+        <update_rate>200</update_rate>
         <imu>
           <angular_velocity>
@@ -69,80 +67,127 @@
           </linear_acceleration>
         </imu>
-    </sensor>
-    <material>Gazebo/Grey</material>
+        <plugin name="turtlebot3_imu" filename="libgazebo_ros_imu_sensor.so">
+          <ros>
+            <!-- <namespace>/tb3</namespace> -->
+            <remapping>~/out:=$(arg prefix)imu</remapping>
+          </ros>
+        </plugin>
+      </sensor>
+      <material>Gazebo/Grey</material>
   </gazebo>
  <gazebo>
-    <plugin
-      filename="libgz-sim-diff-drive-system.so"
-      name="gz::sim::systems::DiffDrive">
+    <plugin name="turtlebot3_diff_drive" filename="libgazebo_ros_diff_drive.so">
+      <ros>
+        <!-- <namespace>/tb3</namespace> -->
+      </ros>
+      <update_rate>30</update_rate>
+      <!-- wheels -->
       <left_joint>wheel_left_joint</left_joint>
       <right_joint>wheel_right_joint</right_joint>
-      <wheel_separation>${wheel_separation}</wheel_separation>
-      <wheel_radius>0.033</wheel_radius>
-      <child_frame_id>$(arg prefix)base_footprint</child_frame_id>
+      <!-- kinematics -->
+      <wheel_separation>0.287</wheel_separation>
+      <wheel_diameter>0.066</wheel_diameter>
+      <!-- limits -->
+      <max_wheel_torque>20</max_wheel_torque>
+      <max_wheel_acceleration>1.0</max_wheel_acceleration>
+      <command_topic>$(arg prefix)cmd_vel</command_topic>
+      <!-- output -->
+      <publish_odom>true</publish_odom>
+      <publish_odom_tf>true</publish_odom_tf>
+      <publish_wheel_tf>false</publish_wheel_tf>
+      <odometry_topic>$(arg prefix)odom</odometry_topic>
+      <odometry_frame>$(arg prefix)odom</odometry_frame>
+      <robot_base_frame>$(arg prefix)base_footprint</robot_base_frame>
     </plugin>
 </gazebo>
   <gazebo reference="$(arg prefix)base_scan">
     <material>Gazebo/FlatBlack</material>
-    <sensor type="gpu_ray" name="lds_lfcd_sensor">
-<!--       <pose>0 0 0 0 0 0</pose> -->
-      <update_rate>5</update_rate>
-      <topic>$(arg prefix)scan</topic>
-      <gz_frame_id>$(arg prefix)base_scan</gz_frame_id>
-      <ray>
-        <scan>
-          <horizontal>
-            <samples>360</samples>
-            <resolution>1</resolution>
-            <min_angle>0.0</min_angle>
-            <max_angle>6.28319</max_angle>
-          </horizontal>
-        </scan>
-        <range>
-          <min>0.120</min>
-          <max>3.5</max>
-          <resolution>0.015</resolution>
-        </range>
-        <noise>
-          <type>gaussian</type>
-          <mean>0.0</mean>
-          <stddev>0.01</stddev>
-        </noise>
-      </ray>
-    </sensor>
+<sensor name="hls_lfcd_lds" type="ray">
+        <always_on>true</always_on>
+        <visualize>true</visualize>
+        <pose>-0.064 0 0.121 0 0 0</pose>
+        <update_rate>5</update_rate>
+        <ray>
+          <scan>
+            <horizontal>
+              <samples>360</samples>
+              <resolution>1.000000</resolution>
+              <min_angle>0.000000</min_angle>
+              <max_angle>6.280000</max_angle>
+            </horizontal>
+          </scan>
+          <range>
+            <min>0.120000</min>
+            <max>3.5</max>
+            <resolution>0.015000</resolution>
+          </range>
+          <noise>
+            <type>gaussian</type>
+            <mean>0.0</mean>
+            <stddev>0.01</stddev>
+          </noise>
+        </ray>
+        <plugin name="turtlebot3_laserscan" filename="libgazebo_ros_ray_sensor.so">
+          <ros>
+            <!-- <namespace>/tb3</namespace> -->
+            <remapping>~/out:=$(arg prefix)scan</remapping>
+          </ros>
+          <output_type>sensor_msgs/LaserScan</output_type>
+          <frame_name>$(arg prefix)base_scan</frame_name>
+        </plugin>
+      </sensor>
   </gazebo>
 <!--link : https://www.raspberrypi.org/documentation/hardware/camera/-->
   <xacro:if value="$(arg use_cam)">
   <gazebo reference="$(arg prefix)camera_rgb_frame">
-    <sensor type="camera" name="pi_camera">
-      <always_on>true</always_on>
-      <camera>
-        <optical_frame_id>$(arg prefix)camera_rgb_optical_frame</optical_frame_id>
-          <horizontal_fov>1.085595</horizontal_fov>
-          <image>
-              <width>640</width>
-              <height>480</height>
-              <format>R8G8B8</format>
-          </image>
-          <clip>
-              <near>0.03</near>
-              <far>100</far>
-          </clip>
+        <sensor type="camera" name="camera1">
+      <update_rate>30.0</update_rate>
+      <camera name="head">
+        <horizontal_fov>1.3962634</horizontal_fov>
+        <image>
+          <width>800</width>
+          <height>800</height>
+          <format>R8G8B8</format>
+        </image>
+        <clip>
+          <near>0.02</near>
+          <far>300</far>
+        </clip>
+        <noise>
+          <type>gaussian</type>
+          <!-- Noise is sampled independently per pixel on each frame.
+               That pixel's noise value is added to each of its color
+               channels, which at that point lie in the range [0,1]. -->
+          <mean>0.0</mean>
+          <stddev>0.007</stddev>
+        </noise>
       </camera>
-       <topic>$(arg prefix)image</topic>
-      <enable_metrics>false</enable_metrics>
+      <plugin name="camera_controller" filename="libgazebo_ros_camera.so">
+        <alwaysOn>true</alwaysOn>
+        <updateRate>0.0</updateRate>
+        <cameraName>rrbot/camera1</cameraName>
+        <imageTopicName>image_raw</imageTopicName>
+        <cameraInfoTopicName>camera_info</cameraInfoTopicName>
+        <frameName>$(arg prefix)camera_rgb_frame</frameName>
+        <hackBaseline>0.07</hackBaseline>
+        <distortionK1>0.0</distortionK1>
+        <distortionK2>0.0</distortionK2>
+        <distortionK3>0.0</distortionK3>
+        <distortionT1>0.0</distortionT1>
+        <distortionT2>0.0</distortionT2>
+      </plugin>
     </sensor>
   </gazebo>
 </xacro:if>
    <gazebo>
-      <plugin filename="libignition-gazebo-joint-state-publisher-system.so" name="ignition::gazebo::systems::JointStatePublisher"/>
-      <plugin
-            filename="ignition-gazebo-pose-publisher-system"
-            name="ignition::gazebo::systems::PosePublisher">
-            <publish_link_pose>false</publish_link_pose>
-            <publish_collision_pose>false</publish_collision_pose>
-            <publish_visual_pose>false</publish_visual_pose>
-            <publish_nested_model_pose>true</publish_nested_model_pose>
-        </plugin>
+    <plugin name="turtlebot3_joint_state" filename="libgazebo_ros_joint_state_publisher.so">
+      <ros>
+        <!-- <namespace>/tb3</namespace> -->
+        <remapping>~/out:=$(arg prefix)joint_states</remapping>
+      </ros>
+      <update_rate>30</update_rate>
+      <joint_name>wheel_left_joint</joint_name>
+      <joint_name>wheel_right_joint</joint_name>
+    </plugin>
     </gazebo>
 </robot>
