Commit message: Tags and Depth in main ws

File: install/turtlebot3_gazebo/share/turtlebot3_gazebo/urdf/my_bot.urdf (robot description, URDF)
Before this commit: robot turtlebot3_waffle_pi, 11 links, 10 joints
Links:
- removed link bot_1/base_footprint
- removed link bot_1/base_link
- removed link bot_1/base_scan
- removed link bot_1/camera_link
- removed link bot_1/camera_rgb_frame
- removed link bot_1/camera_rgb_optical_frame
- removed link bot_1/caster_back_left_link
- removed link bot_1/caster_back_right_link
- removed link bot_1/imu_link
- removed link bot_1/wheel_left_link
- removed link bot_1/wheel_right_link
- added link bot_0/base_footprint
- added link bot_0/base_link, mass 1.3729096e+00; collision box size=0.266 0.266 0.094; visual mesh filename=file:///home/duck_sh/Mobile-Swarm-Navigation/install/turtle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 scale=0.001 0.001 0.001
- added link bot_0/base_scan, mass 0.114; collision cylinder length=0.0315 radius=0.055; visual mesh filename=file:///home/duck_sh/Mobile-Swarm-Navigation/install/turtle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 scale=0.001 0.001 0.001
- added link bot_0/camera_depth_frame
- added link bot_0/camera_link; collision box size=0.015 0.030 0.027
- added link bot_0/camera_rgb_depth_frame
- added link bot_0/camera_rgb_frame
- added link bot_0/camera_rgb_optical_frame
- added link bot_0/caster_back_left_link, mass 0.005; collision sphere radius=0.009
- added link bot_0/caster_back_right_link, mass 0.005; collision sphere radius=0.009
- added link bot_0/imu_link, mass 0.001
- added link bot_0/marker_1; collision box size=0.1 0.1 0.0001; visual mesh filename=package://turtlebot3_xacro/meshes/markers/april_1.dae scale=0.1 0.1 0.1
- added link bot_0/marker_2; collision box size=0.1 0.1 0.0001; visual mesh filename=package://turtlebot3_xacro/meshes/markers/april_2.dae scale=0.1 0.1 0.1
- added link bot_0/marker_3; collision box size=0.1 0.1 0.0001; visual mesh filename=package://turtlebot3_xacro/meshes/markers/april_3.dae scale=0.1 0.1 0.1
- added link bot_0/marker_4; collision box size=0.1 0.1 0.0001; visual mesh filename=package://turtlebot3_xacro/meshes/markers/april_4.dae scale=0.1 0.1 0.1
- added link bot_0/wheel_left_link, mass 2.8498940e-02; collision cylinder length=0.018 radius=0.033; visual mesh filename=file:///home/duck_sh/Mobile-Swarm-Navigation/install/turtle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 scale=0.001 0.001 0.001
- added link bot_0/wheel_right_link, mass 2.8498940e-02; collision cylinder length=0.018 radius=0.033; visual mesh filename=file:///home/duck_sh/Mobile-Swarm-Navigation/install/turtle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 scale=0.001 0.001 0.001
Joints:
- added joint camera_depth_joint: type fixed, parent bot_0/camera_link, child bot_0/camera_depth_frame, origin xyz=0.003 0.011 0.009 rpy=0 0 0
- added joint camera_rgb_depth_joint: type fixed, parent bot_0/camera_depth_frame, child bot_0/camera_rgb_depth_frame, origin xyz=0 0 0 rpy=-1.57 0 -1.57
- added joint marker_joint_1: type fixed, parent bot_0/base_link, child bot_0/marker_1, origin xyz=-0.1 0.134 0.05 rpy=-1.57 3.14 0
- added joint marker_joint_2: type fixed, parent bot_0/base_link, child bot_0/marker_2, origin xyz=-0.1 -0.134 0.05 rpy=1.57 0 0
- added joint marker_joint_3: type fixed, parent bot_0/base_link, child bot_0/marker_3, origin xyz=0.074 0 0.05 rpy=1.57 0 1.57
- added joint marker_joint_4: type fixed, parent bot_0/base_link, child bot_0/marker_4, origin xyz=-0.194 -0 0.05 rpy=1.57 0 -1.57
- joint base_joint: child bot_1/base_link -> bot_0/base_link; parent bot_1/base_footprint -> bot_0/base_footprint
- joint camera_joint: child bot_1/camera_link -> bot_0/camera_link; parent bot_1/base_link -> bot_0/base_link
- joint camera_rgb_joint: child bot_1/camera_rgb_frame -> bot_0/camera_rgb_frame; parent bot_1/camera_link -> bot_0/camera_link
- joint camera_rgb_optical_joint: child bot_1/camera_rgb_optical_frame -> bot_0/camera_rgb_optical_frame; parent bot_1/camera_rgb_frame -> bot_0/camera_rgb_frame
- joint caster_back_left_joint: child bot_1/caster_back_left_link -> bot_0/caster_back_left_link; parent bot_1/base_link -> bot_0/base_link
- joint caster_back_right_joint: child bot_1/caster_back_right_link -> bot_0/caster_back_right_link; parent bot_1/base_link -> bot_0/base_link
- joint imu_joint: child bot_1/imu_link -> bot_0/imu_link; parent bot_1/base_link -> bot_0/base_link
- joint scan_joint: child bot_1/base_scan -> bot_0/base_scan; parent bot_1/base_link -> bot_0/base_link
- joint wheel_left_joint: child bot_1/wheel_left_link -> bot_0/wheel_left_link; parent bot_1/base_link -> bot_0/base_link
- joint wheel_right_joint: child bot_1/wheel_right_link -> bot_0/wheel_right_link; parent bot_1/base_link -> bot_0/base_link

File: install/turtlebot3_gazebo/share/turtlebot3_gazebo/urdf/turtlebot3_waffle_pi.xacro (robot description, xacro)
@@ -1 +1,169 @@
-/home/pacman/turtlebot3_ws/src/turtlebot3/turtlebot3_simulations/turtlebot3_gazebo/urdf/turtlebot3_waffle_pi.xacro
+<?xml version="1.0" ?>
+<robot name="turtlebot3_waffle_pi" xmlns:xacro="http://ros.org/wiki/xacro">
+  <!-- Define the robot_namespace parameter with a default value (empty string) -->
+  <xacro:arg name='robot_namespace' default=''/>
+  <!-- Init colours -->
+  <material name="black">
+      <color rgba="0.0 0.0 0.0 1.0"/>
+  </material>
+  <material name="dark">
+    <color rgba="0.3 0.3 0.3 1.0"/>
+  </material>
+  <material name="light_black">
+    <color rgba="0.4 0.4 0.4 1.0"/>
+  </material>
+  <material name="blue">
+    <color rgba="0.0 0.0 0.8 1.0"/>
+  </material>
+  <material name="green">
+    <color rgba="0.0 0.8 0.0 1.0"/>
+  </material>
+  <material name="grey">
+    <color rgba="0.5 0.5 0.5 1.0"/>
+  </material>
+  <material name="orange">
+    <color rgba="1.0 0.4235 0.0392 1.0"/>
+  </material>
+  <material name="brown">
+    <color rgba="0.8706 0.8118 0.7647 1.0"/>
+  </material>
+  <material name="red">
+    <color rgba="0.8 0.0 0.0 1.0"/>
+  </material>
+  <material name="white">
+    <color rgba="1.0 1.0 1.0 1.0"/>
+  </material>
+  <link name="$(arg robot_namespace)/base_footprint"/>
+  <joint name="$(arg robot_namespace)/base_joint" type="fixed">
+    <parent link="$(arg robot_namespace)/base_footprint"/>
+    <child link="$(arg robot_namespace)/base_link"/>
+    <origin xyz="0 0 0.010" rpy="0 0 0"/>
+  </joint>
+  <link name="$(arg robot_namespace)/base_link">
+    <visual>
+      <origin xyz="-0.064 0 0.0" rpy="0 0 0"/>
+      <geometry>
+        <mesh filename="package://turtlebot3_gazebo/models/turtlebot3_common/meshes/waffle_pi_base.dae" scale="0.001 0.001 0.001"/>
+      </geometry>
+      <material name="light_black"/>
+    </visual>
+    <collision>
+      <origin xyz="-0.064 0 0.047" rpy="0 0 0"/>
+      <geometry>
+        <box size="0.266 0.266 0.094"/>
+      </geometry>
+    </collision>
+    <inertial>
+      <origin xyz="0 0 0" rpy="0 0 0"/>
+      <mass value="1.3729096e+00"/>
+      <inertia ixx="8.7002718e-03" ixy="-4.7576583e-05" ixz="1.1160499e-04"
+               iyy="8.6195418e-03" iyz="-3.5422299e-06"
+               izz="1.4612727e-02" />
+    </inertial>
+  </link>
+  <joint name="$(arg robot_namespace)/wheel_left_joint" type="continuous">
+    <parent link="$(arg robot_namespace)/base_link"/>
+    <child link="$(arg robot_namespace)/wheel_left_link"/>
+    <origin xyz="0.0 0.144 0.023" rpy="-1.57 0 0"/>
+    <axis xyz="0 0 1"/>
+  </joint>
+  <link name="$(arg robot_namespace)/wheel_left_link">
+    <visual>
+      <origin xyz="0 0 0" rpy="1.57 0 0"/>
+      <geometry>
+        <mesh filename="package://turtlebot3_gazebo/models/turtlebot3_common/meshes/tire.dae" scale="0.001 0.001 0.001"/>
+      </geometry>
+      <material name="dark"/>
+    </visual>
+    <collision>
+      <origin xyz="0 0 0" rpy="0 0 0"/>
+      <geometry>
+        <cylinder length="0.018" radius="0.033"/>
+      </geometry>
+    </collision>
+    <inertial>
+      <origin xyz="0 0 0" />
+      <mass value="2.8498940e-02" />
+      <inertia ixx="1.1175580e-05" ixy="-4.2369783e-11" ixz="-5.9381719e-09"
+               iyy="1.1192413e-05" iyz="-1.4400107e-11"
+               izz="2.0712558e-05" />
+    </inertial>
+  </link>
+  <joint name="$(arg robot_namespace)/wheel_right_joint" type="continuous">
+    <parent link="$(arg robot_namespace)/base_link"/>
+    <child link="$(arg robot_namespace)/wheel_right_link"/>
+    <origin xyz="0.0 -0.144 0.023" rpy="-1.57 0 0"/>
+    <axis xyz="0 0 1"/>
+  </joint>
+  <link name="$(arg robot_namespace)/wheel_right_link">
+    <visual>
+      <origin xyz="0 0 0" rpy="1.57 0 0"/>
+      <geometry>
+        <mesh filename="package://turtlebot3_gazebo/models/turtlebot3_common/meshes/tire.dae" scale="0.001 0.001 0.001"/>
+      </geometry>
+      <material name="dark"/>
+    </visual>
+    <collision>
+      <origin xyz="0 0 0" rpy="0 0 0"/>
+      <geometry>
+        <cylinder length="0.018" radius="0.033"/>
+      </geometry>
+    </collision>
+    <inertial>
+      <origin xyz="0 0 0" />
+      <mass value="2.8498940e-02" />
+      <inertia ixx="1.1175580e-05" ixy="-4.2369783e-11" ixz="-5.9381719e-09"
+               iyy="1.1192413e-05" iyz="-1.4400107e-11"
+               izz="2.0712558e-05" />
+    </inertial>
+  </link>
+  <joint name="$(arg robot_namespace)/caster_back_right_joint" type="fixed">
+    <parent link="$(arg robot_namespace)/base_link"/>
+    <child link="$(arg robot_namespace)/caster_back_right_link"/>
+    <origin xyz="-0.177 -0.064 -0.004" rpy="-1.57 0 0"/>
+  </joint>
+  <link name="$(arg robot_namespace)/caster_back_right_link">
+    <collision>
+      <origin xyz="0 0.001 0" rpy="0 0 0"/>
+      <geometry>
+        <box size="0.030 0.009 0.020"/>
+      </geometry>
+    </collision>
+    <inertial>
+      <origin xyz="0 0 0" />
+      <mass value="0.005" />
+      <inertia ixx="0.001" ixy="0.0" ixz="0.0"
+               iyy="0.001" iyz="0.0"
+               izz="0.001" />
+    </inertial>
+  </link>
+  <!-- April Tags -->
+  <xacro:macro name="april_marker" params="marker_id xyz rpy">
+    <link name="marker_${marker_id}">
+      <visual name="marker_visual_${marker_id}">
+        <geometry>
+          <mesh filename="package://turtlebot3_manipulation_description/meshes/markers/april_${marker_id}.dae" scale ="0.1 0.1 0.1"/>
+        </geometry>
+        <!-- <material name="aruco_${marker_id}-material" submesh="${marker_id}"/> -->
+          <!-- <texture filename="package://turtlebot3_manipulation_description/meshes/markers/aruco_${marker_id}.png"/> -->
+        <!-- </material> -->
+      </visual>
+      <collision name="marker_collision_${marker_id}">
+        <geometry>
+          <box size="0.1 0.1 0.0001"/>
+        </geometry>
+      </collision>
+    </link>
+    <joint name="marker_joint_${marker_id}" type="fixed">
+      <parent link="$(arg prefix)base_link"/>
+      <child link="marker_${marker_id}"/>
+      <origin xyz="${xyz}" rpy="${rpy}"/>
+    </joint>
+  </xacro:macro>
+  <!-- ArUco marker instances on TurtleBot3 -->
+  <xacro:april_marker marker_id="1" xyz="-0.1 0.134 0.05" rpy="-1.57 3.14 0"/>
+  <xacro:april_marker marker_id="2" xyz="-0.1 -0.134 0.05" rpy="1.57 0 0"/>
+  <xacro:april_marker marker_id="3" xyz="0.074 0 0.05" rpy="1.57 0 1.57"/>
+  <xacro:april_marker marker_id="4" xyz="-0.194 -0 0.05" rpy="1.57 0 -1.57"/>
+  <!-- Add similar $(arg robot_namespace)/ prefix for remaining links and joints -->
+</robot>

File: install/turtlebot3_xacro/share/turtlebot3_xacro/urdf/turtlebot3_gazebo.xacro (robot description, xacro)
@@ -179,5 +179,45 @@
     </sensor>
   </gazebo>
-</xacro:if>
+  <!-- depth_cam -->
+    <gazebo reference="$(arg prefix)camera_depth_frame">
+        <sensor type="depth" name="depth_camera1">
+      <update_rate>30.0</update_rate>
+      <camera name="head_depth">
+        <horizontal_fov>1.3962634</horizontal_fov>
+        <image>
+          <width>800</width>
+          <height>800</height>
+          <format>R8G8B8</format>
+        </image>
+        <clip>
+          <near>0.02</near>
+          <far>300</far>
+        </clip>
+        <noise>
+          <type>gaussian</type>
+          <!-- Noise is sampled independently per pixel on each frame.
+               That pixel's noise value is added to each of its color
+               channels, which at that point lie in the range [0,1]. -->
+          <mean>0.0</mean>
+          <stddev>0.007</stddev>
+        </noise>
+      </camera>
+      <plugin name="depth_camera_controller" filename="libgazebo_ros_camera.so">
+        <alwaysOn>true</alwaysOn>
+        <updateRate>0.0</updateRate>
+        <cameraName>rrbot/depth_camera1</cameraName>
+        <imageTopicName>image_raw</imageTopicName>
+        <cameraInfoTopicName>camera_info</cameraInfoTopicName>
+        <frameName>$(arg prefix)camera_depth_frame</frameName>
+        <hackBaseline>0.07</hackBaseline>
+        <distortionK1>0.0</distortionK1>
+        <distortionK2>0.0</distortionK2>
+        <distortionK3>0.0</distortionK3>
+        <distortionT1>0.0</distortionT1>
+        <distortionT2>0.0</distortionT2>
+      </plugin>
+    </sensor>
+  </gazebo>
+  </xacro:if>
    <gazebo>
     <plugin name="turtlebot3_joint_state" filename="libgazebo_ros_joint_state_publisher.so">

File: install/turtlebot3_xacro/share/turtlebot3_xacro/urdf/turtlebot3_waffle_pi.urdf.xacro (robot description, xacro)
@@ -225,3 +225,45 @@
   </joint>
   <link name="$(arg prefix)camera_rgb_optical_frame"/>
+  <!-- depth cam -->
+    <joint name="camera_depth_joint" type="fixed">
+    <origin xyz="0.003 0.011 0.009" rpy="0 0 0"/>
+    <parent link="$(arg prefix)camera_link"/>
+    <child link="$(arg prefix)camera_depth_frame"/>
+  </joint>
+  <link name="$(arg prefix)camera_depth_frame"/>
+  <joint name="camera_rgb_depth_joint" type="fixed">
+    <origin xyz="0 0 0" rpy="-1.57 0 -1.57"/>
+    <parent link="$(arg prefix)camera_depth_frame"/>
+    <child link="$(arg prefix)camera_rgb_depth_frame"/>
+  </joint>
+  <link name="$(arg prefix)camera_rgb_depth_frame"/>
+<!-- April Tags -->
+  <xacro:macro name="april_marker" params="marker_id xyz rpy">
+    <link name="$(arg prefix)marker_${marker_id}">
+      <visual name="marker_visual_${marker_id}">
+        <geometry>
+          <mesh filename="package://turtlebot3_xacro/meshes/markers/april_${marker_id}.dae" scale ="0.1 0.1 0.1"/>
+        </geometry>
+        <!-- <material name="aruco_${marker_id}-material" submesh="${marker_id}"/> -->
+          <!-- <texture filename="package://turtlebot3_manipulation_description/meshes/markers/aruco_${marker_id}.png"/> -->
+        <!-- </material> -->
+      </visual>
+      <collision name="marker_collision_${marker_id}">
+        <geometry>
+          <box size="0.1 0.1 0.0001"/>
+        </geometry>
+      </collision>
+    </link>
+    <joint name="marker_joint_${marker_id}" type="fixed">
+      <parent link="$(arg prefix)base_link"/>
+      <child link="$(arg prefix)marker_${marker_id}"/>
+      <origin xyz="${xyz}" rpy="${rpy}"/>
+    </joint>
+  </xacro:macro>
+  <!-- ArUco marker instances on TurtleBot3 -->
+  <xacro:april_marker marker_id="1" xyz="-0.1 0.134 0.05" rpy="-1.57 3.14 0"/>
+  <xacro:april_marker marker_id="2" xyz="-0.1 -0.134 0.05" rpy="1.57 0 0"/>
+  <xacro:april_marker marker_id="3" xyz="0.074 0 0.05" rpy="1.57 0 1.57"/>
+  <xacro:april_marker marker_id="4" xyz="-0.194 -0 0.05" rpy="1.57 0 -1.57"/>
+  <!-- Add similar $(arg robot_namespace)/ prefix for remaining links and joints -->
 </robot>

File: src/turtlebot3/turtlebot3_simulations/turtlebot3_gazebo/urdf/turtlebot3_waffle_pi.xacro (robot description, xacro)
@@ -138,4 +138,32 @@
     </inertial>
   </link>
+  <!-- April Tags -->
+  <xacro:macro name="april_marker" params="marker_id xyz rpy">
+    <link name="marker_${marker_id}">
+      <visual name="marker_visual_${marker_id}">
+        <geometry>
+          <mesh filename="package://turtlebot3_manipulation_description/meshes/markers/april_${marker_id}.dae" scale ="0.1 0.1 0.1"/>
+        </geometry>
+        <!-- <material name="aruco_${marker_id}-material" submesh="${marker_id}"/> -->
+          <!-- <texture filename="package://turtlebot3_manipulation_description/meshes/markers/aruco_${marker_id}.png"/> -->
+        <!-- </material> -->
+      </visual>
+      <collision name="marker_collision_${marker_id}">
+        <geometry>
+          <box size="0.1 0.1 0.0001"/>
+        </geometry>
+      </collision>
+    </link>
+    <joint name="marker_joint_${marker_id}" type="fixed">
+      <parent link="$(arg prefix)base_link"/>
+      <child link="marker_${marker_id}"/>
+      <origin xyz="${xyz}" rpy="${rpy}"/>
+    </joint>
+  </xacro:macro>
+  <!-- ArUco marker instances on TurtleBot3 -->
+  <xacro:april_marker marker_id="1" xyz="-0.1 0.134 0.05" rpy="-1.57 3.14 0"/>
+  <xacro:april_marker marker_id="2" xyz="-0.1 -0.134 0.05" rpy="1.57 0 0"/>
+  <xacro:april_marker marker_id="3" xyz="0.074 0 0.05" rpy="1.57 0 1.57"/>
+  <xacro:april_marker marker_id="4" xyz="-0.194 -0 0.05" rpy="1.57 0 -1.57"/>
   <!-- Add similar $(arg robot_namespace)/ prefix for remaining links and joints -->
 </robot>

File: src/turtlebot3_xacro/urdf/turtlebot3_gazebo.xacro (robot description, xacro)
@@ -179,5 +179,45 @@
     </sensor>
   </gazebo>
-</xacro:if>
+  <!-- depth_cam -->
+    <gazebo reference="$(arg prefix)camera_depth_frame">
+        <sensor type="depth" name="depth_camera1">
+      <update_rate>30.0</update_rate>
+      <camera name="head_depth">
+        <horizontal_fov>1.3962634</horizontal_fov>
+        <image>
+          <width>800</width>
+          <height>800</height>
+          <format>R8G8B8</format>
+        </image>
+        <clip>
+          <near>0.02</near>
+          <far>300</far>
+        </clip>
+        <noise>
+          <type>gaussian</type>
+          <!-- Noise is sampled independently per pixel on each frame.
+               That pixel's noise value is added to each of its color
+               channels, which at that point lie in the range [0,1]. -->
+          <mean>0.0</mean>
+          <stddev>0.007</stddev>
+        </noise>
+      </camera>
+      <plugin name="depth_camera_controller" filename="libgazebo_ros_camera.so">
+        <alwaysOn>true</alwaysOn>
+        <updateRate>0.0</updateRate>
+        <cameraName>rrbot/depth_camera1</cameraName>
+        <imageTopicName>image_raw</imageTopicName>
+        <cameraInfoTopicName>camera_info</cameraInfoTopicName>
+        <frameName>$(arg prefix)camera_depth_frame</frameName>
+        <hackBaseline>0.07</hackBaseline>
+        <distortionK1>0.0</distortionK1>
+        <distortionK2>0.0</distortionK2>
+        <distortionK3>0.0</distortionK3>
+        <distortionT1>0.0</distortionT1>
+        <distortionT2>0.0</distortionT2>
+      </plugin>
+    </sensor>
+  </gazebo>
+  </xacro:if>
    <gazebo>
     <plugin name="turtlebot3_joint_state" filename="libgazebo_ros_joint_state_publisher.so">
