Commit message: In progress arm merging

File: install/turtlebot3_xacro/share/turtlebot3_xacro/urdf/common_properties.xacro (robot description, xacro)
@@ -32,8 +32,8 @@
     <color rgba="1.0 1.0 1.0 1.0"/>
   </material>
- <xacro:arg name="gazebo" default="true"/>
+ <!-- <xacro:arg name="gazebo" default="true"/>
  <xacro:if value="$(arg gazebo)">
    <xacro:include filename="$(find turtlebot3_xacro)/urdf/turtlebot3_gazebo.xacro"/>
- </xacro:if>
+ </xacro:if> -->
  <xacro:macro name="mesh" params="mesh">
      <mesh filename="file://$(find turtlebot3_xacro)/meshes/${mesh}" scale="0.001 0.001 0.001"/>

File: install/turtlebot3_xacro/share/turtlebot3_xacro/urdf/turtlebot3_gazebo.xacro (robot description, xacro)
@@ -1,25 +1,21 @@
 <?xml version="1.0"?>
 <robot name="turtlebot3_gazebo" xmlns:xacro="http://ros.org/wiki/xacro">
-<!-- Arguments common to all turtlebots -->
- <xacro:arg name="prefix"    default=""/>
- <xacro:arg name="cmd_vel_topic"    default="cmd_vel"/>
- <xacro:arg name="odom_topic"    default="odom"/>
- <xacro:arg name="publish_odom"    default="false"/>
-<gazebo reference="$(arg prefix)base_link">
+<xacro:macro name="turtlebot3_gazebo" params="prefix">
+<gazebo reference="${prefix}base_link">
   <material>Gazebo/DarkGrey</material>
 </gazebo>
-<gazebo reference="$(arg prefix)wheel_left_link">
-  <material>Gazebo/FlatBlack</material>
-</gazebo>
-<gazebo reference="$(arg prefix)wheel_right_link">
-  <material>Gazebo/FlatBlack</material>
-</gazebo>
-<gazebo reference="$(arg prefix)caster_back_right_link">
-  <material>Gazebo/FlatBlack</material>
-</gazebo>
-<gazebo reference="$(arg prefix)caster_back_left_link">
-  <material>Gazebo/FlatBlack</material>
-</gazebo>
-  <gazebo reference="$(arg prefix)imu_link">
+<gazebo reference="${prefix}wheel_left_link">
+  <material>Gazebo/FlatBlack</material>
+</gazebo>
+<gazebo reference="${prefix}wheel_right_link">
+  <material>Gazebo/FlatBlack</material>
+</gazebo>
+<gazebo reference="${prefix}caster_back_right_link">
+  <material>Gazebo/FlatBlack</material>
+</gazebo>
+<gazebo reference="${prefix}caster_back_left_link">
+  <material>Gazebo/FlatBlack</material>
+</gazebo>
+  <gazebo reference="${prefix}imu_link">
     <sensor name="tb3_imu" type="imu">
         <always_on>true</always_on>
@@ -70,5 +66,5 @@
           <ros>
             <!-- <namespace>/tb3</namespace> -->
-            <remapping>~/out:=$(arg prefix)imu</remapping>
+            <remapping>~/out:=${prefix}imu</remapping>
           </ros>
         </plugin>
@@ -91,15 +87,15 @@
       <max_wheel_torque>20</max_wheel_torque>
       <max_wheel_acceleration>1.0</max_wheel_acceleration>
-      <command_topic>$(arg prefix)cmd_vel</command_topic>
+      <command_topic>${prefix}cmd_vel</command_topic>
       <!-- output -->
       <publish_odom>true</publish_odom>
       <publish_odom_tf>true</publish_odom_tf>
       <publish_wheel_tf>false</publish_wheel_tf>
-      <odometry_topic>$(arg prefix)odom</odometry_topic>
-      <odometry_frame>$(arg prefix)odom</odometry_frame>
-      <robot_base_frame>$(arg prefix)base_footprint</robot_base_frame>
+      <odometry_topic>${prefix}odom</odometry_topic>
+      <odometry_frame>${prefix}odom</odometry_frame>
+      <robot_base_frame>${prefix}base_footprint</robot_base_frame>
     </plugin>
 </gazebo>
-  <gazebo reference="$(arg prefix)base_scan">
+  <gazebo reference="${prefix}base_scan">
     <material>Gazebo/FlatBlack</material>
 <sensor name="hls_lfcd_lds" type="ray">
@@ -131,14 +127,13 @@
           <ros>
             <!-- <namespace>/tb3</namespace> -->
-            <remapping>~/out:=$(arg prefix)scan</remapping>
+            <remapping>~/out:=${prefix}scan</remapping>
           </ros>
           <output_type>sensor_msgs/LaserScan</output_type>
-          <frame_name>$(arg prefix)base_scan</frame_name>
+          <frame_name>${prefix}base_scan</frame_name>
         </plugin>
       </sensor>
   </gazebo>
 <!--link : https://www.raspberrypi.org/documentation/hardware/camera/-->
-  <xacro:if value="$(arg use_cam)">
-  <gazebo reference="$(arg prefix)camera_rgb_frame">
+  <gazebo reference="${prefix}camera_rgb_frame">
         <sensor type="camera" name="camera1">
       <update_rate>30.0</update_rate>
@@ -169,5 +164,5 @@
         <imageTopicName>image_raw</imageTopicName>
         <cameraInfoTopicName>camera_info</cameraInfoTopicName>
-        <frameName>$(arg prefix)camera_rgb_frame</frameName>
+        <frameName>${prefix}camera_rgb_frame</frameName>
         <hackBaseline>0.07</hackBaseline>
         <distortionK1>0.0</distortionK1>
@@ -180,5 +175,5 @@
   </gazebo>
   <!-- depth_cam -->
-    <gazebo reference="$(arg prefix)camera_depth_frame">
+    <gazebo reference="${prefix}camera_depth_frame">
         <sensor type="depth" name="depth_camera1">
       <update_rate>30.0</update_rate>
@@ -209,5 +204,10 @@
         <imageTopicName>image_raw</imageTopicName>
         <cameraInfoTopicName>camera_info</cameraInfoTopicName>
-        <frameName>$(arg prefix)camera_depth_frame</frameName>
+        <depthImageTopicName>/depth/image_raw</depthImageTopicName>
+        <depthImageCameraInfoTopicName>/depth/camera_info</depthImageCameraInfoTopicName>
+        <pointCloudTopicName>depth_cloud</pointCloudTopicName>
+        <frameName>${prefix}camera_depth_frame</frameName>
+        <pointCloudCutoff>0.5</pointCloudCutoff>
+        <pointCloudCutoffMax>3.5</pointCloudCutoffMax>
         <hackBaseline>0.07</hackBaseline>
         <distortionK1>0.0</distortionK1>
@@ -219,10 +219,9 @@
     </sensor>
   </gazebo>
-  </xacro:if>
    <gazebo>
     <plugin name="turtlebot3_joint_state" filename="libgazebo_ros_joint_state_publisher.so">
       <ros>
         <!-- <namespace>/tb3</namespace> -->
-        <remapping>~/out:=$(arg prefix)joint_states</remapping>
+        <remapping>~/out:=${prefix}joint_states</remapping>
       </ros>
       <update_rate>30</update_rate>
@@ -231,3 +230,4 @@
     </plugin>
     </gazebo>
+</xacro:macro>
 </robot>

File: install/turtlebot3_xacro/share/turtlebot3_xacro/urdf/turtlebot3_waffle_pi.urdf.xacro (robot description, xacro)
@@ -1,15 +1,15 @@
 <?xml version="1.0" ?>
 <robot name="turtlebot3_waffle_pi" xmlns:xacro="http://ros.org/wiki/xacro">
+ <xacro:macro name="turtlebot3_waffle_pi" params="prefix">
  <!-- Properties of waffle_pi -->
  <xacro:property name="wheel_separation" value="0.287" />
- <xacro:arg name="use_cam"    default="true"/>
  <xacro:include filename="$(find turtlebot3_xacro)/urdf/common_properties.urdf"/>
- <link name="$(arg prefix)base_footprint"/>
+ <link name="${prefix}base_footprint"/>
   <joint name="base_joint" type="fixed">
-    <parent link="$(arg prefix)base_footprint"/>
-    <child link="$(arg prefix)base_link" />
+    <parent link="${prefix}base_footprint"/>
+    <child link="${prefix}base_link" />
     <origin xyz="0 0 0.010" rpy="0 0 0"/>
   </joint>
-  <link name="$(arg prefix)base_link">
+  <link name="${prefix}base_link">
     <visual>
       <origin xyz="-0.064 0 0.0" rpy="0 0 0"/>
@@ -33,11 +33,11 @@
   </link>
   <joint name="wheel_left_joint" type="continuous">
-    <parent link="$(arg prefix)base_link"/>
-    <child link="$(arg prefix)wheel_left_link"/>
+    <parent link="${prefix}base_link"/>
+    <child link="${prefix}wheel_left_link"/>
     <origin xyz="0.0 0.144 0.023" rpy="-1.57 0 0"/>
     <axis xyz="0 0 1"/>
     <limit velocity="7.88" effort="10"/>
   </joint>
-  <link name="$(arg prefix)wheel_left_link">
+  <link name="${prefix}wheel_left_link">
     <visual>
       <origin xyz="0 0 0" rpy="1.57 0 0"/>
@@ -69,11 +69,11 @@
   </link>
   <joint name="wheel_right_joint" type="continuous">
-    <parent link="$(arg prefix)base_link"/>
-    <child link="$(arg prefix)wheel_right_link"/>
+    <parent link="${prefix}base_link"/>
+    <child link="${prefix}wheel_right_link"/>
     <origin xyz="0.0 -0.144 0.023" rpy="-1.57 0 0"/>
     <axis xyz="0 0 1"/>
     <limit velocity="7.88" effort="10"/>
   </joint>
-  <link name="$(arg prefix)wheel_right_link">
+  <link name="${prefix}wheel_right_link">
     <visual>
       <origin xyz="0 0 0" rpy="1.57 0 0"/>
@@ -105,9 +105,9 @@
   </link>
   <joint name="caster_back_right_joint" type="fixed">
-    <parent link="$(arg prefix)base_link"/>
-    <child link="$(arg prefix)caster_back_right_link"/>
+    <parent link="${prefix}base_link"/>
+    <child link="${prefix}caster_back_right_link"/>
     <origin xyz="-0.177 -0.064 -0.004" rpy="-1.57 0 0"/>
   </joint>
-  <link name="$(arg prefix)caster_back_right_link">
+  <link name="${prefix}caster_back_right_link">
     <collision>
       <origin xyz="0 0.001 0" rpy="0 0 0"/>
@@ -134,9 +134,9 @@
   </link>
   <joint name="caster_back_left_joint" type="fixed">
-    <parent link="$(arg prefix)base_link"/>
-    <child link="$(arg prefix)caster_back_left_link"/>
+    <parent link="${prefix}base_link"/>
+    <child link="${prefix}caster_back_left_link"/>
     <origin xyz="-0.177 0.064 -0.004" rpy="-1.57 0 0"/>
   </joint>
-  <link name="$(arg prefix)caster_back_left_link">
+  <link name="${prefix}caster_back_left_link">
     <collision>
       <origin xyz="0 0.001 0" rpy="0 0 0"/>
@@ -163,9 +163,9 @@
   </link>
   <joint name="imu_joint" type="fixed">
-    <parent link="$(arg prefix)base_link"/>
-    <child link="$(arg prefix)imu_link"/>
+    <parent link="${prefix}base_link"/>
+    <child link="${prefix}imu_link"/>
     <origin xyz="0.0 0 0.068" rpy="0 0 0"/>
   </joint>
-  <link name="$(arg prefix)imu_link">
+  <link name="${prefix}imu_link">
         <inertial>
       <mass value="0.001"/>
@@ -174,9 +174,9 @@
   </link>
   <joint name="scan_joint" type="fixed">
-    <parent link="$(arg prefix)base_link"/>
-    <child link="$(arg prefix)base_scan"/>
+    <parent link="${prefix}base_link"/>
+    <child link="${prefix}base_scan"/>
     <origin xyz="-0.064 0 0.122" rpy="0 0 0"/>
   </joint>
-  <link name="$(arg prefix)base_scan">
+  <link name="${prefix}base_scan">
     <visual>
       <origin xyz="0 0 0.0" rpy="0 0 0"/>
@@ -202,8 +202,8 @@
   <joint name="camera_joint" type="fixed">
     <origin xyz="0.073 -0.011 0.084" rpy="0 0 0"/>
-    <parent link="$(arg prefix)base_link"/>
-    <child link="$(arg prefix)camera_link"/>
-  </joint>
-  <link name="$(arg prefix)camera_link">
+    <parent link="${prefix}base_link"/>
+    <child link="${prefix}camera_link"/>
+  </joint>
+  <link name="${prefix}camera_link">
     <collision>
       <origin xyz="0.005 0.011 0.013" rpy="0 0 0"/>
@@ -215,30 +215,30 @@
   <joint name="camera_rgb_joint" type="fixed">
     <origin xyz="0.003 0.011 0.009" rpy="0 0 0"/>
-    <parent link="$(arg prefix)camera_link"/>
-    <child link="$(arg prefix)camera_rgb_frame"/>
-  </joint>
-  <link name="$(arg prefix)camera_rgb_frame"/>
+    <parent link="${prefix}camera_link"/>
+    <child link="${prefix}camera_rgb_frame"/>
+  </joint>
+  <link name="${prefix}camera_rgb_frame"/>
   <joint name="camera_rgb_optical_joint" type="fixed">
     <origin xyz="0 0 0" rpy="-1.57 0 -1.57"/>
-    <parent link="$(arg prefix)camera_rgb_frame"/>
-    <child link="$(arg prefix)camera_rgb_optical_frame"/>
-  </joint>
-  <link name="$(arg prefix)camera_rgb_optical_frame"/>
+    <parent link="${prefix}camera_rgb_frame"/>
+    <child link="${prefix}camera_rgb_optical_frame"/>
+  </joint>
+  <link name="${prefix}camera_rgb_optical_frame"/>
   <!-- depth cam -->
     <joint name="camera_depth_joint" type="fixed">
     <origin xyz="0.003 0.011 0.009" rpy="0 0 0"/>
-    <parent link="$(arg prefix)camera_link"/>
-    <child link="$(arg prefix)camera_depth_frame"/>
-  </joint>
-  <link name="$(arg prefix)camera_depth_frame"/>
+    <parent link="${prefix}camera_link"/>
+    <child link="${prefix}camera_depth_frame"/>
+  </joint>
+  <link name="${prefix}camera_depth_frame"/>
   <joint name="camera_rgb_depth_joint" type="fixed">
     <origin xyz="0 0 0" rpy="-1.57 0 -1.57"/>
-    <parent link="$(arg prefix)camera_depth_frame"/>
-    <child link="$(arg prefix)camera_rgb_depth_frame"/>
-  </joint>
-  <link name="$(arg prefix)camera_rgb_depth_frame"/>
+    <parent link="${prefix}camera_depth_frame"/>
+    <child link="${prefix}camera_rgb_depth_frame"/>
+  </joint>
+  <link name="${prefix}camera_rgb_depth_frame"/>
 <!-- April Tags -->
   <xacro:macro name="april_marker" params="marker_id xyz rpy">
-    <link name="$(arg prefix)marker_${marker_id}">
+    <link name="${prefix}marker_${marker_id}">
       <visual name="marker_visual_${marker_id}">
         <geometry>
@@ -256,6 +256,6 @@
     </link>
     <joint name="marker_joint_${marker_id}" type="fixed">
-      <parent link="$(arg prefix)base_link"/>
-      <child link="$(arg prefix)marker_${marker_id}"/>
+      <parent link="${prefix}base_link"/>
+      <child link="${prefix}marker_${marker_id}"/>
       <origin xyz="${xyz}" rpy="${rpy}"/>
     </joint>
@@ -267,3 +267,4 @@
   <xacro:april_marker marker_id="4" xyz="-0.194 -0 0.05" rpy="1.57 0 -1.57"/>
   <!-- Add similar $(arg robot_namespace)/ prefix for remaining links and joints -->
+</xacro:macro>
 </robot>

File: src/turtlebot3_xacro/urdf/turtlebot3_gazebo.xacro (robot description, xacro)
@@ -1,26 +1,22 @@
 <?xml version="1.0"?>
-<robot name="turtlebot3_gazebo" xmlns:xacro="http://ros.org/wiki/xacro">
-<!-- Arguments common to all turtlebots -->
- <xacro:arg name="prefix"    default=""/>
- <xacro:arg name="cmd_vel_topic"    default="cmd_vel"/>
- <xacro:arg name="odom_topic"    default="odom"/>
- <xacro:arg name="publish_odom"    default="false"/>
-<gazebo reference="$(arg prefix)base_link">
-  <material>Gazebo/DarkGrey</material>
-</gazebo>
-<gazebo reference="$(arg prefix)wheel_left_link">
-  <material>Gazebo/FlatBlack</material>
-</gazebo>
-<gazebo reference="$(arg prefix)wheel_right_link">
-  <material>Gazebo/FlatBlack</material>
-</gazebo>
-<gazebo reference="$(arg prefix)caster_back_right_link">
-  <material>Gazebo/FlatBlack</material>
-</gazebo>
-<gazebo reference="$(arg prefix)caster_back_left_link">
-  <material>Gazebo/FlatBlack</material>
-</gazebo>
-  <gazebo reference="$(arg prefix)imu_link">
-    <sensor name="tb3_imu" type="imu">
+<robot xmlns:xacro="http://ros.org/wiki/xacro">
+  <xacro:macro name="turtlebot3_gazebo" params="prefix">
+    <gazebo reference="${prefix}base_link">
+      <material>Gazebo/DarkGrey</material>
+    </gazebo>
+    <gazebo reference="${prefix}wheel_left_link">
+      <material>Gazebo/FlatBlack</material>
+    </gazebo>
+    <gazebo reference="${prefix}wheel_right_link">
+      <material>Gazebo/FlatBlack</material>
+    </gazebo>
+    <gazebo reference="${prefix}caster_back_right_link">
+      <material>Gazebo/FlatBlack</material>
+    </gazebo>
+    <gazebo reference="${prefix}caster_back_left_link">
+      <material>Gazebo/FlatBlack</material>
+    </gazebo>
+    <gazebo reference="${prefix}imu_link">
+      <sensor name="tb3_imu" type="imu">
         <always_on>true</always_on>
         <update_rate>200</update_rate>
@@ -70,5 +66,5 @@
           <ros>
             <!-- <namespace>/tb3</namespace> -->
-            <remapping>~/out:=$(arg prefix)imu</remapping>
+            <remapping>~/out:=${prefix}imu</remapping>
           </ros>
         </plugin>
@@ -91,17 +87,17 @@
       <max_wheel_torque>20</max_wheel_torque>
       <max_wheel_acceleration>1.0</max_wheel_acceleration>
-      <command_topic>$(arg prefix)cmd_vel</command_topic>
+      <command_topic>${prefix}cmd_vel</command_topic>
       <!-- output -->
       <publish_odom>true</publish_odom>
       <publish_odom_tf>true</publish_odom_tf>
       <publish_wheel_tf>false</publish_wheel_tf>
-      <odometry_topic>$(arg prefix)odom</odometry_topic>
-      <odometry_frame>$(arg prefix)odom</odometry_frame>
-      <robot_base_frame>$(arg prefix)base_footprint</robot_base_frame>
+      <odometry_topic>${prefix}odom</odometry_topic>
+      <odometry_frame>${prefix}odom</odometry_frame>
+      <robot_base_frame>${prefix}base_footprint</robot_base_frame>
     </plugin>
 </gazebo>
-  <gazebo reference="$(arg prefix)base_scan">
+  <gazebo reference="${prefix}base_scan">
     <material>Gazebo/FlatBlack</material>
-<sensor name="hls_lfcd_lds" type="ray">
+      <sensor name="hls_lfcd_lds" type="ray">
         <always_on>true</always_on>
         <visualize>true</visualize>
@@ -131,14 +127,13 @@
           <ros>
             <!-- <namespace>/tb3</namespace> -->
-            <remapping>~/out:=$(arg prefix)scan</remapping>
+            <remapping>~/out:=${prefix}scan</remapping>
           </ros>
           <output_type>sensor_msgs/LaserScan</output_type>
-          <frame_name>$(arg prefix)base_scan</frame_name>
+          <frame_name>${prefix}base_scan</frame_name>
         </plugin>
       </sensor>
   </gazebo>
 <!--link : https://www.raspberrypi.org/documentation/hardware/camera/-->
-  <xacro:if value="$(arg use_cam)">
-  <gazebo reference="$(arg prefix)camera_rgb_frame">
+  <gazebo reference="${prefix}camera_rgb_frame">
         <sensor type="camera" name="camera1">
       <update_rate>30.0</update_rate>
@@ -169,5 +164,5 @@
         <imageTopicName>image_raw</imageTopicName>
         <cameraInfoTopicName>camera_info</cameraInfoTopicName>
-        <frameName>$(arg prefix)camera_rgb_frame</frameName>
+        <frameName>${prefix}camera_rgb_frame</frameName>
         <hackBaseline>0.07</hackBaseline>
         <distortionK1>0.0</distortionK1>
@@ -180,5 +175,5 @@
   </gazebo>
   <!-- depth_cam -->
-    <gazebo reference="$(arg prefix)camera_depth_frame">
+    <gazebo reference="${prefix}camera_depth_frame">
         <sensor type="depth" name="depth_camera1">
       <update_rate>30.0</update_rate>
@@ -209,5 +204,10 @@
         <imageTopicName>image_raw</imageTopicName>
         <cameraInfoTopicName>camera_info</cameraInfoTopicName>
-        <frameName>$(arg prefix)camera_depth_frame</frameName>
+        <depthImageTopicName>/depth/image_raw</depthImageTopicName>
+        <depthImageCameraInfoTopicName>/depth/camera_info</depthImageCameraInfoTopicName>
+        <pointCloudTopicName>depth_cloud</pointCloudTopicName>
+        <frameName>${prefix}camera_depth_frame</frameName>
+        <pointCloudCutoff>0.5</pointCloudCutoff>
+        <pointCloudCutoffMax>3.5</pointCloudCutoffMax>
         <hackBaseline>0.07</hackBaseline>
         <distortionK1>0.0</distortionK1>
@@ -219,10 +219,9 @@
     </sensor>
   </gazebo>
-  </xacro:if>
    <gazebo>
     <plugin name="turtlebot3_joint_state" filename="libgazebo_ros_joint_state_publisher.so">
       <ros>
         <!-- <namespace>/tb3</namespace> -->
-        <remapping>~/out:=$(arg prefix)joint_states</remapping>
+        <remapping>~/out:=${prefix}joint_states</remapping>
       </ros>
       <update_rate>30</update_rate>
@@ -231,3 +230,4 @@
     </plugin>
     </gazebo>
+</xacro:macro>
 </robot>

File: src/turtlebot3_xacro/urdf/turtlebot3_waffle_pi.urdf.xacro (robot description, xacro)
@@ -3,5 +3,4 @@
  <!-- Properties of waffle_pi -->
  <xacro:property name="wheel_separation" value="0.287" />
- <xacro:arg name="use_cam"    default="true"/>
  <xacro:include filename="$(find turtlebot3_xacro)/urdf/common_properties.urdf"/>
  <link name="$(arg prefix)base_footprint"/>
@@ -225,45 +224,3 @@
   </joint>
   <link name="$(arg prefix)camera_rgb_optical_frame"/>
-  <!-- depth cam -->
-    <joint name="camera_depth_joint" type="fixed">
-    <origin xyz="0.003 0.011 0.009" rpy="0 0 0"/>
-    <parent link="$(arg prefix)camera_link"/>
-    <child link="$(arg prefix)camera_depth_frame"/>
-  </joint>
-  <link name="$(arg prefix)camera_depth_frame"/>
-  <joint name="camera_rgb_depth_joint" type="fixed">
-    <origin xyz="0 0 0" rpy="-1.57 0 -1.57"/>
-    <parent link="$(arg prefix)camera_depth_frame"/>
-    <child link="$(arg prefix)camera_rgb_depth_frame"/>
-  </joint>
-  <link name="$(arg prefix)camera_rgb_depth_frame"/>
-<!-- April Tags -->
-  <xacro:macro name="april_marker" params="marker_id xyz rpy">
-    <link name="$(arg prefix)marker_${marker_id}">
-      <visual name="marker_visual_${marker_id}">
-        <geometry>
-          <mesh filename="package://turtlebot3_xacro/meshes/markers/april_${marker_id}.dae" scale ="0.1 0.1 0.1"/>
-        </geometry>
-        <!-- <material name="aruco_${marker_id}-material" submesh="${marker_id}"/> -->
-          <!-- <texture filename="package://turtlebot3_manipulation_description/meshes/markers/aruco_${marker_id}.png"/> -->
-        <!-- </material> -->
-      </visual>
-      <collision name="marker_collision_${marker_id}">
-        <geometry>
-          <box size="0.1 0.1 0.0001"/>
-        </geometry>
-      </collision>
-    </link>
-    <joint name="marker_joint_${marker_id}" type="fixed">
-      <parent link="$(arg prefix)base_link"/>
-      <child link="$(arg prefix)marker_${marker_id}"/>
-      <origin xyz="${xyz}" rpy="${rpy}"/>
-    </joint>
-  </xacro:macro>
-  <!-- ArUco marker instances on TurtleBot3 -->
-  <xacro:april_marker marker_id="1" xyz="-0.1 0.134 0.05" rpy="-1.57 3.14 0"/>
-  <xacro:april_marker marker_id="2" xyz="-0.1 -0.134 0.05" rpy="1.57 0 0"/>
-  <xacro:april_marker marker_id="3" xyz="0.074 0 0.05" rpy="1.57 0 1.57"/>
-  <xacro:april_marker marker_id="4" xyz="-0.194 -0 0.05" rpy="1.57 0 -1.57"/>
-  <!-- Add similar $(arg robot_namespace)/ prefix for remaining links and joints -->
 </robot>
