Commit message: started semantic map

File: src/turtlebot3_xacro/urdf/turtlebot3_gazebo.xacro (robot description, xacro)
@@ -21,4 +21,8 @@
   <material>Gazebo/FlatBlack</material>
 </gazebo>
+<gazebo reference="$(arg prefix)april_marker_1"/>
+<gazebo reference="$(arg prefix)april_marker_2"/>
+<gazebo reference="$(arg prefix)april_marker_3"/>
+<gazebo reference="$(arg prefix)april_marker_4"/>
   <gazebo reference="$(arg prefix)imu_link">
     <sensor name="tb3_imu" type="imu">
@@ -70,5 +74,6 @@
           <ros>
             <!-- <namespace>/tb3</namespace> -->
-            <remapping>~/out:=$(arg prefix)imu</remapping>
+            <!-- <remapping>~/out:=$(arg prefix)imu</remapping> -->
+            <remapping>~/out:=imu</remapping>
           </ros>
         </plugin>
@@ -131,5 +136,6 @@
           <ros>
             <!-- <namespace>/tb3</namespace> -->
-            <remapping>~/out:=$(arg prefix)scan</remapping>
+            <!-- <remapping>~/out:=$(arg prefix)scan</remapping> -->
+            <remapping>~/out:=scan</remapping>
           </ros>
           <output_type>sensor_msgs/LaserScan</output_type>
@@ -140,6 +146,47 @@
 <!--link : https://www.raspberrypi.org/documentation/hardware/camera/-->
   <xacro:if value="$(arg use_cam)">
+    <gazebo reference="$(arg prefix)camera_rgb_frame">
+        <sensor type="depth" name="camera1">
+        <update_rate>30.0</update_rate>
+        <visualize>true</visualize>
+        <camera name="head">
+            <horizontal_fov>1.3962634</horizontal_fov>
+            <image>
+            <width>800</width>
+            <height>800</height>
+            <format>R8G8B8</format>
+            </image>
+            <clip>
+            <near>0.02</near>
+            <far>300</far>
+            </clip>
+            <noise>
+            <type>gaussian</type>
+            <!-- Noise is sampled independently per pixel on each frame.
+                That pixel's noise value is added to each of its color
+                channels, which at that point lie in the range [0,1]. -->
+            <mean>0.0</mean>
+            <stddev>0.007</stddev>
+            </noise>
+        </camera>
+        <plugin name="depth_camera_controller" filename="libgazebo_ros_camera.so">
+            <alwaysOn>true</alwaysOn>
+            <updateRate>0.0</updateRate>
+            <cameraName>rrbot/camera1</cameraName>
+            <depthImageTopicName>image_raw</depthImageTopicName>
+            <cameraInfoTopicName>camera_info</cameraInfoTopicName>
+            <pointCloudTopicName>points</pointCloudTopicName>
+            <frame_name>$(arg prefix)camera_rgb_depth_frame</frame_name>
+            <hackBaseline>0.07</hackBaseline>
+            <distortionK1>0.0</distortionK1>
+            <distortionK2>0.0</distortionK2>
+            <distortionK3>0.0</distortionK3>
+            <distortionT1>0.0</distortionT1>
+            <distortionT2>0.0</distortionT2>
+        </plugin>
+        </sensor>
+  </gazebo>
   <gazebo reference="$(arg prefix)camera_rgb_frame">
-        <sensor type="camera" name="camera1">
+        <sensor type="camera" name="camera2">
       <update_rate>30.0</update_rate>
       <camera name="head">
@@ -166,5 +213,5 @@
         <alwaysOn>true</alwaysOn>
         <updateRate>0.0</updateRate>
-        <cameraName>rrbot/camera1</cameraName>
+        <cameraName>rrbot/camera2</cameraName>
         <imageTopicName>image_raw</imageTopicName>
         <cameraInfoTopicName>camera_info</cameraInfoTopicName>

File: src/turtlebot3_xacro/urdf/turtlebot3_waffle_pi.urdf.xacro (robot description, xacro)
@@ -4,5 +4,5 @@
  <xacro:property name="wheel_separation" value="0.287" />
  <xacro:arg name="use_cam"    default="true"/>
- <xacro:include filename="$(find turtlebot3_xacro)/urdf/common_properties.urdf"/>
+ <xacro:include filename="$(find turtlebot3_xacro)/urdf/common_properties.xacro"/>
  <link name="$(arg prefix)base_footprint"/>
   <joint name="base_joint" type="fixed">
@@ -225,3 +225,45 @@
   </joint>
   <link name="$(arg prefix)camera_rgb_optical_frame"/>
+  <!-- depth cam -->
+    <joint name="camera_depth_joint" type="fixed">
+    <origin xyz="0.003 0.011 0.009" rpy="0 0 0"/>
+    <parent link="$(arg prefix)camera_link"/>
+    <child link="$(arg prefix)camera_depth_frame"/>
+  </joint>
+  <link name="$(arg prefix)camera_depth_frame"/>
+  <joint name="camera_rgb_depth_joint" type="fixed">
+    <origin xyz="0 0 0" rpy="-1.57 0 -1.57"/>
+    <parent link="$(arg prefix)camera_depth_frame"/>
+    <child link="$(arg prefix)camera_rgb_depth_frame"/>
+  </joint>
+  <link name="$(arg prefix)camera_rgb_depth_frame"/>
+<!-- April Tags -->
+  <xacro:macro name="april_marker" params="marker_id xyz rpy">
+    <link name="$(arg prefix)marker_${marker_id}">
+      <visual name="marker_visual_${marker_id}">
+        <geometry>
+          <xacro:mesh mesh="markers/april_${marker_id}.dae" />
+        </geometry>
+        <!-- <material name="aruco_${marker_id}-material" submesh="${marker_id}"/> -->
+          <!-- <texture filename="package://turtlebot3_manipulation_description/meshes/markers/aruco_${marker_id}.png"/> -->
+        <!-- </material> -->
+      </visual>
+      <collision name="marker_collision_${marker_id}">
+        <geometry>
+          <box size="0.1 0.1 0.0001"/>
+        </geometry>
+      </collision>
+    </link>
+    <joint name="marker_joint_${marker_id}" type="fixed">
+      <parent link="$(arg prefix)base_link"/>
+      <child link="$(arg prefix)marker_${marker_id}"/>
+      <origin xyz="${xyz}" rpy="${rpy}"/>
+    </joint>
+  </xacro:macro>
+  <!-- ArUco marker instances on TurtleBot3 -->
+  <xacro:april_marker marker_id="1" xyz="-0.1 0.134 0.05" rpy="-1.57 3.14 0"/>
+  <xacro:april_marker marker_id="2" xyz="-0.1 -0.134 0.05" rpy="1.57 0 0"/>
+  <xacro:april_marker marker_id="3" xyz="0.074 0 0.05" rpy="1.57 0 1.57"/>
+  <xacro:april_marker marker_id="4" xyz="-0.194 -0 0.05" rpy="1.57 0 -1.57"/>
+  <!-- Add similar $(arg robot_namespace)/ prefix for remaining links and joints -->
 </robot>
