Commit message: backup

File: src/turtlebot3_xacro/urdf/common_properties.xacro (robot description, xacro)
@@ -32,8 +32,8 @@
     <color rgba="1.0 1.0 1.0 1.0"/>
   </material>
- <!-- <xacro:arg name="gazebo" default="true"/>
+ <xacro:arg name="gazebo" default="true"/>
  <xacro:if value="$(arg gazebo)">
    <xacro:include filename="$(find turtlebot3_xacro)/urdf/turtlebot3_gazebo.xacro"/>
- </xacro:if> -->
+ </xacro:if>
  <xacro:macro name="mesh" params="mesh">
      <mesh filename="file://$(find turtlebot3_xacro)/meshes/${mesh}" scale="0.001 0.001 0.001"/>

File: src/turtlebot3_xacro/urdf/open_manipulator_x.gazebo.xacro (robot description, xacro)
@@ -39,10 +39,10 @@
     <material>Gazebo/Red</material>
   </gazebo>
-  <xacro:SimpleTransmission trans="${prefix}trans1" joint="${prefix}joint1" actuator="${prefix}actuator1" />
-  <xacro:SimpleTransmission trans="${prefix}trans2" joint="${prefix}joint2" actuator="${prefix}actuator2" />
-  <xacro:SimpleTransmission trans="${prefix}trans3" joint="${prefix}joint3" actuator="${prefix}actuator3" />
-  <xacro:SimpleTransmission trans="${prefix}trans4" joint="${prefix}joint4" actuator="${prefix}actuator4" />
-  <xacro:SimpleTransmission trans="${prefix}trans5" joint="${prefix}gripper_left_joint" actuator="${prefix}actuator5" />
-  <xacro:SimpleTransmission trans="${prefix}trans6" joint="${prefix}gripper_right_joint" actuator="${prefix}actuator6" />
+  <xacro:SimpleTransmission trans="${prefix}trans1" joint="${prefix}joint1" actuator="${prefix}/actuator1" />
+  <xacro:SimpleTransmission trans="${prefix}trans2" joint="${prefix}joint2" actuator="${prefix}/actuator2" />
+  <xacro:SimpleTransmission trans="${prefix}trans3" joint="${prefix}joint3" actuator="${prefix}/actuator3" />
+  <xacro:SimpleTransmission trans="${prefix}trans4" joint="${prefix}joint4" actuator="${prefix}/actuator4" />
+  <xacro:SimpleTransmission trans="${prefix}trans5" joint="${prefix}gripper_left_joint" actuator="${prefix}/actuator5" />
+  <xacro:SimpleTransmission trans="${prefix}trans6" joint="${prefix}gripper_right_joint" actuator="${prefix}/actuator6" />
   </xacro:macro>
 </robot>

File: src/turtlebot3_xacro/urdf/open_manipulator_x.urdf.xacro (robot description, xacro)
@@ -3,8 +3,8 @@
 <robot xmlns:xacro="http://www.ros.org/wiki/xacro">
   <xacro:macro name="open_manipulator_x" params="prefix">
-    <xacro:include filename="$(find turtlebot3_xacro)/urdf/common_properties.urdf"/>
+    <!-- <xacro:include filename="$(find turtlebot3_xacro)/urdf/common_properties.urdf"/> -->
     <xacro:property
       name="meshes_file_direction"
-      value="package://turtlebot3_xacro/meshes/open_manipulator_x"/>
+      value="file://$(find turtlebot3_xacro)/meshes/open_manipulator_x"/>
     <link name="${prefix}link1">
       <visual>

File: src/turtlebot3_xacro/urdf/turtlebot3_gazebo_backup.xacro (robot description, xacro)
@@ -1,26 +1,22 @@
 <?xml version="1.0"?>
-<robot name="turtlebot3_gazebo" xmlns:xacro="http://ros.org/wiki/xacro">
-<!-- Arguments common to all turtlebots -->
- <!-- <xacro:arg name="prefix"    default=""/> -->
- <!-- <xacro:arg name="cmd_vel_topic"    default="cmd_vel"/> -->
- <!-- <xacro:arg name="odom_topic"    default="odom"/> -->
- <!-- <xacro:arg name="publish_odom"    default="false"/> -->
-<gazebo reference="$(arg prefix)base_link">
-  <material>Gazebo/DarkGrey</material>
-</gazebo>
-<gazebo reference="$(arg prefix)wheel_left_link">
-  <material>Gazebo/FlatBlack</material>
-</gazebo>
-<gazebo reference="$(arg prefix)wheel_right_link">
-  <material>Gazebo/FlatBlack</material>
-</gazebo>
-<gazebo reference="$(arg prefix)caster_back_right_link">
-  <material>Gazebo/FlatBlack</material>
-</gazebo>
-<gazebo reference="$(arg prefix)caster_back_left_link">
-  <material>Gazebo/FlatBlack</material>
-</gazebo>
-  <gazebo reference="$(arg prefix)imu_link">
-    <sensor name="tb3_imu" type="imu">
+<robot xmlns:xacro="http://ros.org/wiki/xacro">
+  <xacro:macro name="turtlebot3_gazebo" params="prefix">
+    <gazebo reference="${prefix}base_link">
+      <material>Gazebo/DarkGrey</material>
+    </gazebo>
+    <gazebo reference="${prefix}wheel_left_link">
+      <material>Gazebo/FlatBlack</material>
+    </gazebo>
+    <gazebo reference="${prefix}wheel_right_link">
+      <material>Gazebo/FlatBlack</material>
+    </gazebo>
+    <gazebo reference="${prefix}caster_back_right_link">
+      <material>Gazebo/FlatBlack</material>
+    </gazebo>
+    <gazebo reference="${prefix}caster_back_left_link">
+      <material>Gazebo/FlatBlack</material>
+    </gazebo>
+    <gazebo reference="${prefix}imu_link">
+      <sensor name="tb3_imu" type="imu">
         <always_on>true</always_on>
         <update_rate>200</update_rate>
@@ -70,5 +66,5 @@
           <ros>
             <!-- <namespace>/tb3</namespace> -->
-            <remapping>~/out:=$(arg prefix)imu</remapping>
+            <remapping>~/out:=${prefix}imu</remapping>
           </ros>
         </plugin>
@@ -91,17 +87,17 @@
       <max_wheel_torque>20</max_wheel_torque>
       <max_wheel_acceleration>1.0</max_wheel_acceleration>
-      <command_topic>$(arg prefix)cmd_vel</command_topic>
+      <command_topic>${prefix}cmd_vel</command_topic>
       <!-- output -->
       <publish_odom>true</publish_odom>
       <publish_odom_tf>true</publish_odom_tf>
       <publish_wheel_tf>false</publish_wheel_tf>
-      <odometry_topic>$(arg prefix)odom</odometry_topic>
-      <odometry_frame>$(arg prefix)odom</odometry_frame>
-      <robot_base_frame>$(arg prefix)base_footprint</robot_base_frame>
+      <odometry_topic>${prefix}odom</odometry_topic>
+      <odometry_frame>${prefix}odom</odometry_frame>
+      <robot_base_frame>${prefix}base_footprint</robot_base_frame>
     </plugin>
 </gazebo>
-  <gazebo reference="$(arg prefix)base_scan">
+  <gazebo reference="${prefix}base_scan">
     <material>Gazebo/FlatBlack</material>
-<sensor name="hls_lfcd_lds" type="ray">
+      <sensor name="hls_lfcd_lds" type="ray">
         <always_on>true</always_on>
         <visualize>true</visualize>
@@ -131,14 +127,13 @@
           <ros>
             <!-- <namespace>/tb3</namespace> -->
-            <remapping>~/out:=$(arg prefix)scan</remapping>
+            <remapping>~/out:=${prefix}scan</remapping>
           </ros>
           <output_type>sensor_msgs/LaserScan</output_type>
-          <frame_name>$(arg prefix)base_scan</frame_name>
+          <frame_name>${prefix}base_scan</frame_name>
         </plugin>
       </sensor>
   </gazebo>
 <!--link : https://www.raspberrypi.org/documentation/hardware/camera/-->
-  <xacro:if value="$(arg use_cam)">
-  <gazebo reference="$(arg prefix)camera_rgb_frame">
+  <gazebo reference="${prefix}camera_rgb_frame">
         <sensor type="camera" name="camera1">
       <update_rate>30.0</update_rate>
@@ -169,5 +164,5 @@
         <imageTopicName>image_raw</imageTopicName>
         <cameraInfoTopicName>camera_info</cameraInfoTopicName>
-        <frameName>$(arg prefix)camera_rgb_frame</frameName>
+        <frameName>${prefix}camera_rgb_frame</frameName>
         <hackBaseline>0.07</hackBaseline>
         <distortionK1>0.0</distortionK1>
@@ -179,10 +174,54 @@
     </sensor>
   </gazebo>
-</xacro:if>
+  <!-- depth_cam -->
+    <gazebo reference="${prefix}camera_depth_frame">
+        <sensor type="depth" name="depth_camera1">
+      <update_rate>30.0</update_rate>
+      <camera name="head_depth">
+        <horizontal_fov>1.3962634</horizontal_fov>
+        <image>
+          <width>800</width>
+          <height>800</height>
+          <format>R8G8B8</format>
+        </image>
+        <clip>
+          <near>0.02</near>
+          <far>300</far>
+        </clip>
+        <noise>
+          <type>gaussian</type>
+          <!-- Noise is sampled independently per pixel on each frame.
+               That pixel's noise value is added to each of its color
+               channels, which at that point lie in the range [0,1]. -->
+          <mean>0.0</mean>
+          <stddev>0.007</stddev>
+        </noise>
+      </camera>
+      <plugin name="depth_camera_controller" filename="libgazebo_ros_camera.so">
+        <alwaysOn>true</alwaysOn>
+        <updateRate>0.0</updateRate>
+        <cameraName>rrbot/depth_camera1</cameraName>
+        <imageTopicName>image_raw</imageTopicName>
+        <cameraInfoTopicName>camera_info</cameraInfoTopicName>
+        <depthImageTopicName>/depth/image_raw</depthImageTopicName>
+        <depthImageCameraInfoTopicName>/depth/camera_info</depthImageCameraInfoTopicName>
+        <pointCloudTopicName>depth_cloud</pointCloudTopicName>
+        <frameName>${prefix}camera_depth_frame</frameName>
+        <pointCloudCutoff>0.5</pointCloudCutoff>
+        <pointCloudCutoffMax>3.5</pointCloudCutoffMax>
+        <hackBaseline>0.07</hackBaseline>
+        <distortionK1>0.0</distortionK1>
+        <distortionK2>0.0</distortionK2>
+        <distortionK3>0.0</distortionK3>
+        <distortionT1>0.0</distortionT1>
+        <distortionT2>0.0</distortionT2>
+      </plugin>
+    </sensor>
+  </gazebo>
    <gazebo>
     <plugin name="turtlebot3_joint_state" filename="libgazebo_ros_joint_state_publisher.so">
       <ros>
         <!-- <namespace>/tb3</namespace> -->
-        <remapping>~/out:=$(arg prefix)joint_states</remapping>
+        <remapping>~/out:=${prefix}joint_states</remapping>
       </ros>
       <update_rate>30</update_rate>
@@ -191,3 +230,4 @@
     </plugin>
     </gazebo>
+</xacro:macro>
 </robot>

File: src/turtlebot3_xacro/urdf/turtlebot3_manipulation.urdf.xacro (robot description, xacro)
@@ -12,32 +12,30 @@
   <!-- <xacro:arg name="fake_sensor_commands" default="true" /> -->
   <!-- Import common_properties macro -->
-  <!-- <xacro:include filename="$(find turtlebot3_xacro)/urdf/common_properties.xacro" /> -->
+  <xacro:include filename="$(find turtlebot3_xacro)/urdf/common_properties.xacro" />
   <!-- Include TurtleBot3 Waffle Pi urdf macro -->
   <xacro:include filename="$(find turtlebot3_xacro)/urdf/turtlebot3_waffle_pi.urdf.xacro" />
   <!-- Include TurtleBot3 Waffle Pi gazebo macro -->
-  <xacro:include filename="$(find turtlebot3_xacro)/urdf/turtlebot3_gazebo.xacro"/>
+  <xacro:if value="$(arg gazebo)">
+    <!-- <xacro:include filename="$(find turtlebot3_xacro)/urdf/turtlebot3_gazebo.xacro"/> -->
+  </xacro:if>
   <!-- Include OpenManipulator-X urdf macro -->
-  <!-- <xacro:include filename="$(find turtlebot3_xacro)/urdf/open_manipulator_x.urdf.xacro" /> -->
+  <xacro:include filename="$(find turtlebot3_xacro)/urdf/open_manipulator_x.urdf.xacro" />
   <!-- Include OpenManipulator-X gazebo macro -->
-  <!-- <xacro:include filename="$(find turtlebot3_xacro)/urdf/open_manipulator_x.gazebo.xacro" /> -->
+  <xacro:include filename="$(find turtlebot3_xacro)/urdf/open_manipulator_x.gazebo.xacro" />
   <!-- Include TurtleBot3 Manipulation ros2 control macro -->
-  <!-- <xacro:include filename="$(find turtlebot3_xacro)/urdf/turtlebot3_manipulation_system.ros2_control.xacro" /> -->
-  <xacro:turtlebot3_gazebo prefix="$(arg prefix)" />
+  <xacro:include filename="$(find turtlebot3_xacro)/urdf/turtlebot3_manipulation_system.ros2_control.xacro" />
   <!-- Used for fixing OpenManipulator-X on TurtleBot3 Waffle Pi -->
-  <!-- <joint name="$(arg prefix)base_fixed" type="fixed">
+  <joint name="$(arg prefix)base_fixed" type="fixed">
     <parent link="$(arg prefix)base_link"/>
     <child link="$(arg prefix)link1"/>
     <origin xyz="-0.092 0.0 0.091" rpy="0 0 0"/>
-  </joint> -->
-  <!-- <xacro:open_manipulator_x prefix="$(arg prefix)" /> -->
-  <!-- <xacro:open_manipulator_x_gazebo prefix="$(arg prefix)" /> -->
-  <!-- <xacro:turtlebot3_manipulation_system
-    prefix="$(arg prefix)" use_sim="$(arg use_sim)"
-    use_fake_hardware="$(arg use_fake_hardware)"
-    fake_sensor_commands="$(arg fake_sensor_commands)"/> -->
-  <!-- <gazebo>
+  </joint>
+<!--  -->
+  <xacro:open_manipulator_x prefix="$(arg prefix)" />
+  <xacro:open_manipulator_x_gazebo prefix="$(arg prefix)" />
+  <gazebo>
     <plugin name="gazebo_ros2_control" filename="libgazebo_ros2_control.so">
       <parameters>$(find turtlebot3_xacro)/config/gazebo_controller_manager.yaml</parameters>
     </plugin>
-  </gazebo> -->
+  </gazebo>
 </robot>

File: src/turtlebot3_xacro/urdf/turtlebot3_manipulation_system.ros2_control.xacro (robot description, xacro)
@@ -6,5 +6,5 @@
         <plugin>gazebo_ros2_control/GazeboSystem</plugin>
       </hardware>
-      <joint name="${prefix}wheel_left_joint">
+      <!-- <joint name="${prefix}wheel_left_joint">
         <command_interface name="velocity">
           <param name="min">-24.5</param>
@@ -29,6 +29,6 @@
           <param name="initial_value">0.0</param>
         </state_interface>
-      </joint>
-      <sensor name="imu">
+      </joint> -->
+      <!-- <sensor name="imu">
         <state_interface name="orientation.x">
           <param name="initial_value">0.0</param>
@@ -61,6 +61,6 @@
           <param name="initial_value">0.0</param>
         </state_interface>
-      </sensor>
-      <sensor name="battery">
+      </sensor> -->
+      <!-- <sensor name="battery">
         <state_interface name="voltage">
           <param name="initial_value">0.0</param>
@@ -75,5 +75,5 @@
           <param name="initial_value">0.0</param>
         </state_interface>
-      </sensor>
+      </sensor> -->
       <joint name="${prefix}joint1">
         <command_interface name="position">

File: src/turtlebot3_xacro/urdf/turtlebot3_waffle_pi.urdf_backup.xacro (robot description, xacro)
@@ -3,6 +3,5 @@
  <!-- Properties of waffle_pi -->
  <xacro:property name="wheel_separation" value="0.287" />
- <!-- <xacro:arg name="use_cam"    default="true"/> -->
- <!-- <xacro:include filename="$(find turtlebot3_xacro)/urdf/common_properties.urdf"/> -->
+ <xacro:include filename="$(find turtlebot3_xacro)/urdf/common_properties.urdf"/>
  <link name="$(arg prefix)base_footprint"/>
   <joint name="base_joint" type="fixed">
